File: GameCube.kicad_pcb (KiCad board)
At the start: 4 copper layers, 173 x 231.6 mm, 175 parts, among them J1 Conn_02x16_Odd_Even, J2 Conn_02x21_Odd_Even, SW1 SW_Push, SW10 SW_Push, SW11 SW_Push, SW12 SW_Push, SW13 SW_Push, SW14 SW_Push, SW15 SW_Push, SW16 SW_Push, SW17 SW_Push, SW18 SW_Push, SW19 SW_Push, SW2 SW_Push, SW20 SW_Push, SW21 SW_Push, SW22 SW_Push, SW23 SW_Push, SW24 SW_Push, SW25 SW_Push, SW26 SW_Push, SW27 SW_Push, SW28 SW_Push, SW29 SW_Push, SW3 SW_Push, SW30 SW_Push, SW31 SW_Push, SW32 SW_Push, SW33 SW_Push, SW34 SW_Push, SW35 SW_Push, SW36 SW_Push, SW37 SW_Push, SW38 SW_Push, SW39 SW_Push, SW4 SW_Push, SW40 SW_Push, SW41 SW_Push, SW42 SW_Push, SW43 SW_Push, SW44 SW_Push, SW45 SW_Push, SW46 SW_Push, SW47 SW_Push, SW48 SW_Push, SW49 SW_Push, SW5 SW_Push, SW50 SW_Push, SW51 SW_Push, SW52 SW_Push, SW53 SW_Push, SW54 SW_Push, SW6 SW_Push, SW7 SW_Push, SW8 SW_Push, SW9 SW_Push

Commit message: Changed PCB & Schematic Alignment
Parts:
- moved C1 259.6 mm to (32.0, 293.0)
- moved BT2 158.2 mm to (44.0, 325.3)
- moved J1 134.2 mm to (111.7, -9.62)
- moved J2 134.2 mm to (118.0, -40.0)
- moved R5 134.0 mm to (117.8, -33.8)
- moved R9 134.0 mm to (128.3, -33.8)
- moved R1 134.0 mm to (107.9, -33.8)
- moved R2 134.0 mm to (110.5, -33.8)
- moved R3 134.0 mm to (113.0, -33.8)
- moved R4 134.0 mm to (115.6, -33.8)
- moved R6 134.0 mm to (120.5, -33.8)
- moved R7 134.0 mm to (123.5, -33.9)
- moved R8 134.0 mm to (125.7, -33.8)
- moved LED2 77.9 mm to (44.0, 17.7)
- moved D1 77.1 mm to (27.8, 28.3)
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Routing:
- net VDD: track 1733.2 -> 0.00 mm, vias 8 -> 0
- net GND: track 941.0 -> 0.00 mm, vias 68 -> 0
- net Column3: track 280.0 -> 0.00 mm, vias 1 -> 0
- net Row11: track 276.0 -> 0.00 mm, vias 2 -> 0
- net Row10: track 258.5 -> 0.00 mm, vias 6 -> 0
- net Column5: track 245.5 -> 0.00 mm, vias 1 -> 0
- net Column4: track 241.2 -> 0.00 mm, vias 1 -> 0
- net Row9: track 234.3 -> 0.00 mm, vias 6 -> 0
- net Row2: track 218.7 -> 0.00 mm, vias 12 -> 0
- net Row8: track 213.6 -> 0.00 mm, vias 6 -> 0
- net Row1: track 196.9 -> 0.00 mm, vias 17 -> 0
- net Row7: track 186.4 -> 0.00 mm, vias 4 -> 0
- net Row0: track 173.6 -> 0.00 mm, vias 15 -> 0
- net Column0: track 169.5 -> 0.00 mm, vias 1 -> 0
- net Row6: track 165.5 -> 0.00 mm, vias 5 -> 0
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- removed copper zone on F.Cu, net GND
Other:
- board size 173 x 231.6 mm -> 179 x 179 mm

Commit message: Additional Spacing Update
Parts:
- added TP1: Jumper, TestPoint:TestPoint_THTPad_1.5x1.5mm_Drill0.7mm, F.Cu at (70.7, 54.8)
- added TP10: Jumper, TestPoint:TestPoint_THTPad_1.5x1.5mm_Drill0.7mm, F.Cu at (130.4, 214.5)
- added TP11: Jumper, TestPoint:TestPoint_THTPad_1.5x1.5mm_Drill0.7mm, F.Cu at (77.4, 237.5)
- added TP2: Jumper, TestPoint:TestPoint_THTPad_1.5x1.5mm_Drill0.7mm, F.Cu at (78.2, 54.8)
- added TP3: Jumper, TestPoint:TestPoint_THTPad_1.5x1.5mm_Drill0.7mm, F.Cu at (130.9, 33.2)
- added TP4: Jumper, TestPoint:TestPoint_THTPad_1.5x1.5mm_Drill0.7mm, F.Cu at (138.1, 33.2)
- added TP5: Jumper, TestPoint:TestPoint_THTPad_1.5x1.5mm_Drill0.7mm, F.Cu at (176.1, 70.7)
- added TP6: Jumper, TestPoint:TestPoint_THTPad_1.5x1.5mm_Drill0.7mm, F.Cu at (131.0, 93.5)
- added TP7: Jumper, TestPoint:TestPoint_THTPad_1.5x1.5mm_Drill0.7mm, F.Cu at (78.3, 114.8)
- added TP8: Jumper, TestPoint:TestPoint_THTPad_1.5x1.5mm_Drill0.7mm, F.Cu at (78.2, 154.5)
- added TP9: Jumper, TestPoint:TestPoint_THTPad_1.5x1.5mm_Drill0.7mm, F.Cu at (130.4, 176.2)
- moved D50 2.65 mm to (110.1, 231.5)
- moved LED46 2.65 mm to (126.0, 199.2)
- moved LED47 2.65 mm to (104.5, 199.2)
- moved LED48 2.65 mm to (83.0, 199.2)
- moved LED49 2.65 mm to (82.9, 220.7)
- moved LED50 2.65 mm to (104.5, 220.7)
- moved LED51 2.65 mm to (126.0, 220.7)
- moved LED52 2.65 mm to (126.5, 242.2)
- moved LED53 2.65 mm to (104.3, 242.2)
- moved LED54 2.65 mm to (82.7, 242.2)
- moved D46 2.65 mm to (131.6, 209.9)
- moved D47 2.65 mm to (110.0, 209.9)
- moved D48 2.65 mm to (88.5, 209.9)
- moved D49 2.65 mm to (88.6, 231.4)
- moved D51 2.65 mm to (131.6, 231.4)
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Connections:
- LED19 pad 4: Net-(LED18-DOUT) -> Net-(LED19-DIN)
- LED28 pad 4: Net-(LED27-DOUT) -> Net-(LED28-DIN)
- LED37 pad 4: Net-(LED36-DOUT) -> Net-(LED37-DIN)
- LED46 pad 4: Net-(LED45-DOUT) -> Net-(LED46-DIN)
- LED54 pad 2: unconnected-(LED54-DOUT-Pad2) -> Net-(LED54-DOUT)
- LED9 pad 2: Net-(LED10-DIN) -> Net-(LED9-DOUT)
Other:
- board size 179 x 179 mm -> 179 x 239.5 mm
