File: GameCube.kicad_sch (KiCad schematic)
At the start: 175 parts, among them J1 Conn_02x16_Odd_Even, J2 Conn_02x21_Odd_Even, SW1 SW_Push, SW10 SW_Push, SW11 SW_Push, SW12 SW_Push, SW13 SW_Push, SW14 SW_Push, SW15 SW_Push, SW16 SW_Push, SW17 SW_Push, SW18 SW_Push, SW19 SW_Push, SW2 SW_Push, SW20 SW_Push, SW21 SW_Push, SW22 SW_Push, SW23 SW_Push, SW24 SW_Push, SW25 SW_Push, SW26 SW_Push, SW27 SW_Push, SW28 SW_Push, SW29 SW_Push, SW3 SW_Push, SW30 SW_Push, SW31 SW_Push, SW32 SW_Push, SW33 SW_Push, SW34 SW_Push, SW35 SW_Push, SW36 SW_Push, SW37 SW_Push, SW38 SW_Push, SW39 SW_Push, SW4 SW_Push, SW40 SW_Push, SW41 SW_Push, SW42 SW_Push, SW43 SW_Push, SW44 SW_Push, SW45 SW_Push, SW46 SW_Push, SW47 SW_Push, SW48 SW_Push, SW49 SW_Push, SW5 SW_Push, SW50 SW_Push, SW51 SW_Push, SW52 SW_Push, SW53 SW_Push, SW54 SW_Push, SW6 SW_Push, SW7 SW_Push, SW8 SW_Push, SW9 SW_Push

Commit message: Changed PCB & Schematic Alignment
Connections:
- net at LED46.4 (DIN): no longer LED45.2 (DOUT)
- net at LED10.4 (DIN): no longer LED9.2 (DOUT)
- net at LED37.4 (DIN): no longer LED36.2 (DOUT)
- net at LED28.4 (DIN): no longer LED27.2 (DOUT)
- net at LED18.2 (DOUT): no longer LED19.4 (DIN)
- no-connect marks 51 -> 61
Changed lines of the file:
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@@
 	)
 	(no_connect
+		(at 476.25 204.47)
+	)
+	(no_connect
 		(at 203.2 184.15)
 	)
@@
 	)
 	(no_connect
+		(at 260.35 212.09)
+	)
+	(no_connect
 		(at 156.21 173.99)
 	)
@@
 	)
 	(no_connect
+		(at 350.52 146.05)
+	)
+	(no_connect
 		(at 156.21 163.83)
 	)
@@
 	)
 	(no_connect
+		(at 260.35 299.72)
+	)
+	(no_connect
+		(at 379.73 153.67)
+	)
+	(no_connect
 		(at 179.07 156.21)
 	)
@@
 	)
 	(no_connect
+		(at 260.35 335.28)
+	)
+	(no_connect
 		(at 203.2 146.05)
 	)
@@
 	)
 	(no_connect
+		(at 355.6 386.08)
+	)
+	(no_connect
 		(at 203.2 148.59)
 	)
@@
 	)
 	(no_connect
+		(at 355.6 420.37)
+	)
+	(no_connect
 		(at 179.07 158.75)
 	)
 	(no_connect
+		(at 119.38 212.09)
+	)
+	(no_connect
+		(at 350.52 233.68)
+	)
+	(no_connect
 		(at 179.07 153.67)
 	)
@@
 	(wire
 		(pts
-			(xy 476.25 204.47) (xy 476.25 233.68)
-		)
-		(stroke
-			(width 0)
-			(type default)
-			(color 109 0 255 1)
-		)
-	)
-	(wire
-		(pts
 			(xy 621.03 288.29) (xy 643.89 288.29)
 		)
@@
 	(wire
 		(pts
-			(xy 355.6 262.89) (xy 345.44 262.89)
+			(xy 351.79 262.89) (xy 345.44 262.89)
 		)
 		(stroke
@@
 	(wire
 		(pts
-			(xy 345.44 233.68) (xy 476.25 233.68)
+			(xy 345.44 233.68) (xy 350.52 233.68)
 		)
 		(stroke
@@
 	(wire
 		(pts
-			(xy 355.6 386.08) (xy 355.6 420.37)
-		)
-		(stroke
-			(width 0)
-			(type default)
-			(color 109 0 255 1)
-		)
-	)
-	(wire
-		(pts
 			(xy 262.89 201.93) (xy 262.89 204.47)
 		)
@@
 	(wire
 		(pts
-			(xy 260.35 299.72) (xy 260.35 335.28)
-		)
-		(stroke
-			(width 0)
-			(type default)
-			(color 109 0 255 1)
-		)
-	)
-	(wire
-		(pts
 			(xy 229.87 194.31) (xy 229.87 186.69)
 		)
@@
 	(wire
 		(pts
-			(xy 355.6 292.1) (xy 355.6 262.89)
+			(xy 351.79 292.1) (xy 351.79 262.89)
 		)
 		(stroke
@@
 	(wire
 		(pts
-			(xy 344.17 146.05) (xy 370.84 146.05)
+			(xy 344.17 146.05) (xy 350.52 146.05)
 		)
 		(stroke
@@
 	(wire
 		(pts
+			(xy 266.7 212.09) (xy 260.35 212.09)
+		)
+		(stroke
+			(width 0)
+			(type default)
+			(color 109 0 255 1)
+		)
+	)
+	(wire
+		(pts
 			(xy 257.81 457.2) (xy 265.43 457.2)
 		)
@@
 	(wire
 		(pts
-			(xy 370.84 153.67) (xy 388.62 153.67)
+			(xy 379.73 153.67) (xy 388.62 153.67)
 		)
 		(stroke
@@
 	(wire
 		(pts
-			(xy 370.84 146.05) (xy 370.84 153.67)
-		)
-		(stroke
-			(width 0)
-			(type default)
-			(color 109 0 255 1)
-		)
-	)
-	(wire
-		(pts
 			(xy 316.23 247.65) (xy 316.23 241.3)
 		)
@@
 	(wire
 		(pts
-			(xy 119.38 212.09) (xy 266.7 212.09)
-		)
-		(stroke
-			(width 0)
-			(type default)
-			(color 109 0 255 1)
-		)
-	)
-	(wire
-		(pts
 			(xy 88.9 190.5) (xy 85.09 190.5)
 		)
@@
 	(wire
 		(pts
-			(xy 345.44 292.1) (xy 355.6 292.1)
+			(xy 345.44 292.1) (xy 351.79 292.1)
 		)
 		(stroke

Commit message: Additional Spacing Update
Parts:
- added TP1, TP10, TP11, TP2, TP3, TP4, TP5, TP6, TP7, TP8, TP9: Jumper, TestPoint:TestPoint_THTPad_1.5x1.5mm_Drill0.7mm, symbol Connector:TestPoint
Connections:
- net at LED46.4 (DIN): now also TP10.1
- net at LED10.4 (DIN): now also TP2.1
- net at LED54.2 (DOUT): now also TP11.1
- net at LED37.4 (DIN): now also TP8.1
- net at LED28.4 (DIN): now also TP6.1
- net at LED36.2 (DOUT): now also TP7.1
- net at LED18.2 (DOUT): now also TP3.1
- net at LED27.2 (DOUT): now also TP5.1
- net at LED45.2 (DOUT): now also TP9.1
- net at LED19.4 (DIN): now also TP4.1
- net at LED9.2 (DOUT): now also TP1.1
- no-connect marks 61 -> 50
